Commit message: marge lidar and cartographer slam add

File: src/amr_big_two_description/urdf/amr_big_two.xacro (robot description, xacro)
@@ -290,4 +290,6 @@
 <link name="back_lidar_link">
 </link>
+<link name="laser_link">
+</link>
 <joint name="Ball 1" type="continuous">
   <origin xyz="0.325 0.018907 -0.131093" rpy="0 0 0"/>
@@ -369,3 +371,8 @@
   <origin xyz="-0.35 0.3 0.06" rpy="0 0 0"/>
 </joint>
+<joint name="laser" type="fixed">
+  <parent link="base_link"/>
+  <child link="laser_link"/>
+  <origin xyz="0.0 0.0 0.06" rpy="0 0 0"/>
+</joint>
 </robot>

Commit message: added IMU to the robot

File: src/amr_big_two_description/urdf/amr_big_two.xacro (robot description, xacro)
@@ -286,10 +286,8 @@
   </collision>
 </link>
-<link name="front_lidar_link">
-</link>
-<link name="back_lidar_link">
-</link>
-<link name="laser_link">
-</link>
+<link name="front_lidar_link"/>
+<link name="back_lidar_link"/>
+<link name="laser_link"/>
+<link name="imu_link"/>
 <joint name="Ball 1" type="continuous">
   <origin xyz="0.325 0.018907 -0.131093" rpy="0 0 0"/>
@@ -366,4 +364,9 @@
   <origin xyz="0.35 -0.25 0.06" rpy="0 0 0"/>
 </joint>
+<joint name="imu" type="fixed">
+  <parent link="base_link"/>
+  <child link="imu_link"/>
+  <origin xyz="0.0 0.0 0.04" rpy="0 0 0"/>
+</joint>
 <joint name="back_lidar_joint" type="fixed">
   <parent link="base_link"/>

File: src/amr_big_two_description/urdf/diff_dr.xacro (robot description, xacro)
@@ -19,4 +19,81 @@
         </plugin>
      </gazebo>
+    <gazebo reference="imu_link">
+     <sensor name="bmb_imu" type="imu">
+      <always_on>true</always_on>
+      <update_rate>100</update_rate>
+      <visualize>true</visualize>
+      <imu>
+        <orientation>
+          <x>
+            <noise type="gaussian">
+              <mean>0.0</mean>
+              <stddev>2e-3</stddev>
+            </noise>
+          </x>
+          <y>
+            <noise type="gaussian">
+              <mean>0.0</mean>
+              <stddev>2e-3</stddev>
+            </noise>
+          </y>
+          <z>
+            <noise type="gaussian">
+              <mean>0.0</mean>
+              <stddev>2e-3</stddev>
+            </noise>
+          </z>
+        </orientation>
+        <angular_velocity>
+          <x>
+            <noise type="gaussian">
+              <mean>0.0</mean>
+              <stddev>2e-4</stddev>
+            </noise>
+          </x>
+          <y>
+            <noise type="gaussian">
+              <mean>0.0</mean>
+              <stddev>2e-4</stddev>
+            </noise>
+          </y>
+          <z>
+            <noise type="gaussian">
+              <mean>0.0</mean>
+              <stddev>2e-4</stddev>
+            </noise>
+          </z>
+        </angular_velocity>
+        <linear_acceleration>
+          <x>
+            <noise type="gaussian">
+              <mean>0.0</mean>
+              <stddev>1.7e-2</stddev>
+            </noise>
+          </x>
+          <y>
+            <noise type="gaussian">
+              <mean>0.0</mean>
+              <stddev>1.7e-2</stddev>
+            </noise>
+          </y>
+          <z>
+            <noise type="gaussian">
+              <mean>0.0</mean>
+              <stddev>1.7e-2</stddev>
+            </noise>
+          </z>
+        </linear_acceleration>
+      </imu>
+      <plugin name="basic_mobile_bot_imu" filename="libgazebo_ros_imu_sensor.so">
+        <initial_orientation_as_reference>false</initial_orientation_as_reference>
+        <ros>
+          <namespace>/imu</namespace>
+          <remapping>~/out:=data</remapping>
+          <frame_name>imu_link</frame_name>
+        </ros>
+      </plugin>
+    </sensor>
+  </gazebo>
      <gazebo reference="front_lidar_link">
         <sensor name="lidar_1" type="ray">

Commit message: depth cam added and local path planner using depth camera

File: src/amr_big_two_description/urdf/amr_big_two.xacro (robot description, xacro)
@@ -5,5 +5,29 @@
 <xacro:include filename="$(find amr_big_two_description)/urdf/amr_big_two.gazebo" />
 <xacro:include filename="$(find amr_big_two_description)/urdf/diff_dr.xacro" />
-<!-- <xacro:include filename="$(find amr_big_two_description)/urdf/model.sdf" /> -->
+<xacro:include filename="$(find amr_big_two_description)/urdf/depth_cam.xacro" />
+<link name="depth_link"/>
+<link name="camera_link"/>
+<!-- <link name='world'/> -->
+<link name='depth_link_optical'/>
+<!-- <joint name="fix_world" type="fixed">
+  <parent link="world"/>
+  <child link="base_link"/>
+  <origin xyz="0.0 0 0" rpy="0 0 0"/>
+</joint>  -->
+<joint name="fix_depth" type="fixed">
+  <parent link="depth_link"/>
+  <child link="depth_link_optical"/>
+  <origin xyz="0 0 0" rpy="-1.57 0 -1.57"/>
+</joint>
+<joint name="depth" type="fixed">
+  <parent link="cam_v1_1"/>
+  <child link="depth_link"/>
+  <origin xyz="0.4 0 0" rpy="0 0 0"/>
+</joint>
+<joint name="camera" type="fixed">
+  <parent link="cam_v1_1"/>
+  <child link="camera_link"/>
+  <origin xyz="0.4 0 0" rpy="0 0 0"/>
+</joint>
 <link name="base_link">
   <inertial>
